File: pk_detect/pk_det.kicad_sch (KiCad schematic)
At the start: 36 parts, among them J102 Conn_01x08_Socket, U105 TL072, U106 TL072

Commit message: change arch
Parts:
- removed C105, C106, C107, C108: 100n, Capacitor_THT:C_Disc_D4.3mm_W1.9mm_P5.00mm, symbol Device:C
- removed C110, C111, C112, C113: C_Polarized_US, Capacitor_THT:CP_Radial_D6.3mm_P2.50mm, symbol Device:C_Polarized_US
- removed D101, D102, D106, D107: BAT51, Diode_THT:D_DO-15_P12.70mm_Horizontal, symbol Device:D_Schottky
- removed D104, D105, D108, D109: D_Schottky, Diode_THT:D_DO-15_P12.70mm_Horizontal, symbol Device:D_Schottky
- removed J102: Conn_01x08_Socket, Connector_Molex:Molex_KK-254_AE-6410-08A_1x08_P2.54mm_Vertical, symbol Connector:Conn_01x08_Socket
- removed R102, R105, R106, R109, R110, R111, R112, R113, R114, R115: 4k7, Resistor_THT:R_Axial_DIN0207_L6.3mm_D2.5mm_P10.16mm_Horizontal, symbol Device:R_US
- removed RV101, RV102, RV103: R_Potentiometer_Trim_US, Potentiometer_THT:Potentiometer_Bourns_3296W_Vertical, symbol Device:R_Potentiometer_Trim_US
- removed U106: TL072, Package_DIP:DIP-8_W7.62mm_LongPads, symbol Amplifier_Operational:TL072
- added C1, C2: 10u, Capacitor_THT:CP_Radial_D6.3mm_P2.50mm, symbol Device:C_Polarized
- added C3, C4: 22p, Capacitor_THT:C_Disc_D4.3mm_W1.9mm_P5.00mm, symbol Device:C
- added J1, J2: Conn_01x04_Socket, Connector_Molex:Molex_KK-254_AE-6410-04A_1x04_P2.54mm_Vertical, symbol Connector:Conn_01x04_Socket
- added Q1, Q2, Q4, Q5: 2N2907, Package_TO_SOT_THT:TO-46-3, symbol Transistor_BJT:Q_PNP_EBC
- added Q3, Q6, Q7: 2N2222, Package_TO_SOT_THT:TO-46-3, symbol Transistor_BJT:Q_NPN_EBC
- added R1, R10, R11, R12, R13, R14, R2, R3, R4, R5, R6, R7, R8, R9: 22k, Resistor_THT:R_Axial_DIN0207_L6.3mm_D2.5mm_P10.16mm_Horizontal, symbol Device:R_US
Connections:
- net +12V: now also J2.1 (Pin_1), Q6.3 (C), Q7.3 (C), R1.1, R12.1, R13.1, R6.1, R8.1
- net -12V: now also C1.2, J2.3 (Pin_3), Q4.3 (C), Q5.3 (C), R3.2, R4.2, R9.2
- net GND: now also J1.2 (Pin_2), J1.4 (Pin_4), J2.2 (Pin_2), J2.4 (Pin_4), R10.2, R11.1, R14.2, R5.2
- new net: C3.1, Q1.1 (E), R8.2
- new net: C3.2, Q4.2 (B), R10.1
- new net: Q2.1 (E), R4.1, R5.1
- new net: C4.1, Q1.3 (C), R9.1
- new net: C1.1, Q2.2 (B), R2.2, R3.1
- new net: Q5.1 (E), Q7.2 (B), R12.2
- new net: C4.2, Q5.2 (B), R11.2
- new net: Q1.2 (B), Q3.3 (C), R1.2
- new net: C2.2, Q3.2 (B), R6.2, R7.1
- new net: Q2.3 (C), R7.2
- new net: Q3.1 (E), R2.1
- new net: Q4.1 (E), Q6.2 (B), R13.2
- new net: Q6.1 (E), Q7.1 (E), R14.1
- new net IN: C2.1, J1.3 (Pin_3)
- new net OUT: J1.1 (Pin_1)
Other:
- moved on the sheet: C103, C104, R103, R104, U105C
