File: mid_only/equalizer.kicad_pcb (KiCad board)
At the start: 2 copper layers, 43.8 x 58.4 mm, 22 parts, among them J1 Conn_01x04_Socket, J2 Conn_01x04_Socket, U105 TL072

Commit message: med ok
Parts:
- removed R1, R2, R3, R4: 47k, Resistor_THT:R_Axial_DIN0207_L6.3mm_D2.5mm_P10.16mm_Horizontal
- moved R103 18.1 mm to (119.4, 64.8)
- moved C116 15.8 mm to (109.3, 70.5), turned to 0 degrees
- moved C103 14.5 mm to (120.0, 50.8), turned to 180 degrees
- moved U105 13.9 mm to (107.3, 54.6)
- moved R115 12.9 mm to (123.8, 71.8), turned to 90 degrees
- moved C104 12.3 mm to (109.2, 66.0), turned to 0 degrees
- moved R112 11.7 mm to (109.2, 75.6), turned to -90 degrees
- moved R104 11.1 mm to (119.4, 78.7)
- moved R114 10.8 mm to (123.8, 48.9), turned to -90 degrees
- moved R111 10.5 mm to (113.7, 75.6), turned to -90 degrees
- moved C117 7.64 mm to (120.0, 47.0), turned to 90 degrees
- moved J2 7.33 mm to (126.4, 83.5)
- moved J1 7.10 mm to (126.4, 36.8)
- moved C115 4.82 mm to (102.9, 57.2), turned to -90 degrees
- moved R113 2.69 mm to (114.3, 36.8)
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Connections:
- RVSWEEP101 pad 1: Net-(R1-Pad2) -> Net-(U105A-+)
- RVSWEEP101 pad 4: Net-(R2-Pad1) -> Net-(U105A-+)
Routing:
- net GND: track 142.3 -> 264.0 mm
- net Net-(R1-Pad2): track 25.5 -> 0.00 mm
- net Net-(U105A-+): track 47.7 -> 28.8 mm
- net Net-(U105C-V+): track 27.0 -> 8.24 mm
- net Net-(C116-Pad1): track 21.7 -> 5.09 mm
- net +12V: track 5.08 -> 21.0 mm
- net Net-(U105C-V-): track 36.0 -> 21.3 mm, vias 2 -> 0
- net Net-(U105B-+): track 46.7 -> 58.0 mm, vias 2 -> 0
- net Net-(R111-Pad1): track 24.4 -> 14.0 mm
- net Net-(R2-Pad1): track 10.3 -> 0.00 mm
- net Net-(U105B--): track 19.7 -> 11.2 mm
- net Net-(C116-Pad2): track 24.4 -> 31.5 mm
- net IN: track 34.3 -> 28.3 mm
- net Net-(U105A--): track 19.8 -> 24.9 mm
- net Net-(R112-Pad2): track 16.1 -> 13.2 mm
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Other:
- board size 43.8 x 58.4 mm -> 35.6 x 58.4 mm

Commit message: v1
Parts:
- added J3: Conn_01x04_Socket, Connector_Molex:Molex_KK-254_AE-6410-04A_1x04_P2.54mm_Vertical, F.Cu at (125.7, 78.5)
- moved R114 19.8 mm to (117.9, 67.8), turned to 90 degrees
- moved C103 10.2 mm to (109.8, 50.5), turned to 0 degrees
- moved R104 5.61 mm to (118.9, 73.2), turned to 180 degrees
- moved R103 5.49 mm to (124.0, 67.8)
- moved R115 4.90 mm to (120.9, 67.8)
- moved C116 2.24 mm to (109.8, 68.3)
- moved J2 2.15 mm to (125.7, 85.6)
- moved C104 1.02 mm to (109.2, 65.0)
- moved R111 0.89 mm to (113.7, 76.5)
- moved R112 0.89 mm to (109.2, 76.5)
- moved U105 0.81 mm to (106.7, 54.1)
- moved RVSWEEP101 0.53 mm to (97.9, 71.1)
Routing:
- net Net-(U105C-V+): track 8.24 -> 24.4 mm
- net Net-(C116-Pad2): track 31.5 -> 16.3 mm
- net Net-(U105C-V-): track 21.3 -> 13.6 mm
- net -12V: track 5.40 -> 13.0 mm
- net Net-(C116-Pad1): track 5.09 -> 9.55 mm
- net GND: track 264.0 -> 268.2 mm, vias 16 -> 15
- net Net-(U105B--): track 11.2 -> 7.12 mm
- net +12V: track 21.0 -> 17.9 mm
- net Net-(U105A--): track 24.9 -> 22.9 mm
- net Net-(U105B-+): track 58.0 -> 56.6 mm
- net Net-(R112-Pad2): track 13.2 -> 12.5 mm
