File: top_bot_only/top_bot.kicad_pcb (KiCad board)
At the start: 2 copper layers, 35.6 x 58.4 mm, 22 parts, among them J1 Conn_01x04_Socket, J2 Conn_01x04_Socket, U106 TL072

Commit message: v1
Parts:
- added J3: Conn_01x04_Socket, Connector_Molex:Molex_KK-254_AE-6410-04A_1x04_P2.54mm_Vertical, F.Cu at (125.7, 85.3)
- moved J2 5.08 mm to (125.7, 78.5)
- moved R103 4.98 mm to (125.2, 73.2)
- moved R109 0.64 mm to (114.3, 85.1)
- moved RVLF101 0.56 mm to (97.8, 71.1)
Routing:
- net GND: track 203.4 -> 194.2 mm, vias 11 -> 9
- net +12V: track 5.56 -> 12.3 mm
- net Net-(U106C-V+): track 11.7 -> 6.31 mm
- net Net-(C105-Pad1): track 25.4 -> 23.6 mm
- net -12V: track 16.2 -> 17.8 mm
- net Net-(U106A-+): track 27.9 -> 26.6 mm
- net Net-(C111-Pad1): track 14.7 -> 13.5 mm
- net Net-(C111-Pad2): track 18.7 -> 17.9 mm
- net OUT: track 70.4 -> 69.8 mm
