File: top_bot_only/top_bot.kicad_sch (KiCad schematic)
At the start: 22 parts, among them J1 Conn_01x04_Socket, J2 Conn_01x04_Socket, U106 TL072

Commit message: v1
Parts:
- added J3: Conn_01x04_Socket, Connector_Molex:Molex_KK-254_AE-6410-04A_1x04_P2.54mm_Vertical, symbol Connector:Conn_01x04_Socket
Connections:
- net +12V: now also J3.1 (Pin_1)
- net -12V: now also J3.3 (Pin_3)
- net GND: now also J3.2 (Pin_2), J3.4 (Pin_4)
