File: vga/vca.kicad_pcb (KiCad board)
At the start: 2 copper layers, 69.6 x 50.2 mm, 43 parts, among them J1 Conn_01x04_Socket, J2 Conn_01x04_Socket, Q1 2N2222, Q10 2N2222, Q11 2N2222, Q12 2N2907, Q13 2N2907, Q3 2N2222, Q4 2N2222, Q5 2N2907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

Commit message: v1
Parts:
- removed D1, D2: 1N4148, Diode_THT:D_DO-35_SOD27_P7.62mm_Horizontal
- added C2: 100n, Capacitor_THT:C_Disc_D4.3mm_W1.9mm_P5.00mm, F.Cu at (177.3, 55.3)
- added C3: 100n, Capacitor_THT:C_Disc_D4.3mm_W1.9mm_P5.00mm, F.Cu at (174.5, 50.3)
- added C4: 100n, Capacitor_THT:C_Disc_D4.3mm_W1.9mm_P5.00mm, F.Cu at (147.3, 62.7)
- added C5: 100n, Capacitor_THT:C_Disc_D4.3mm_W1.9mm_P5.00mm, F.Cu at (147.3, 74.6)
- added J3: Conn_01x04_Socket, Connector_Molex:Molex_KK-254_AE-6410-04A_1x04_P2.54mm_Vertical, F.Cu at (209.0, 80.5)
- added Q14: 2N2222, Package_TO_SOT_THT:TO-46-3, F.Cu at (201.4, 56.9)
- added Q2: 2N2222, Package_TO_SOT_THT:TO-46-3, F.Cu at (195.6, 53.3)
- moved R8 8.25 mm to (180.3, 50.8)
- moved J2 6.58 mm to (209.0, 69.3)
- moved R9 6.19 mm to (202.2, 61.2)
- moved R3 5.11 mm to (171.4, 55.1)
- moved Q1 3.42 mm to (156.5, 51.6), turned to -90 degrees
- moved R12 3.05 mm to (151.6, 57.1)
- moved Q13 2.93 mm to (179.1, 69.3)
- moved R16 2.92 mm to (154.9, 57.1)
- moved R103 2.69 mm to (183.6, 71.6)
- moved R104 2.67 mm to (183.6, 75.6)
- moved Q7 2.64 mm to (161.3, 71.8)
- moved R1 2.54 mm to (161.3, 50.8)
- moved J1 2.24 mm to (208.8, 64.8)
- moved Q10 2.19 mm to (169.2, 71.8)
- moved Q11 2.16 mm to (169.2, 65.8)
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Connections:
- H1 pad 1: (no net) -> GND
- H2 pad 1: (no net) -> GND
- H3 pad 1: (no net) -> GND
- H4 pad 1: (no net) -> GND
Routing:
- net GND: track 110.3 -> 149.2 mm, vias 41 -> 35
- net -12V: track 115.2 -> 141.3 mm
- net +12V: track 112.9 -> 131.7 mm
- net Net-(U105A--): track 20.3 -> 10.6 mm
- net Net-(Q11-B): track 34.9 -> 28.4 mm
- net Net-(Q10-B): track 41.6 -> 45.8 mm
- net Net-(Q10-C): track 18.9 -> 16.7 mm
- net Net-(U105C-V-): track 8.98 -> 6.86 mm
- net Net-(Q1-B): track 32.1 -> 34.2 mm
- net OUT: track 57.7 -> 59.8 mm
- net Net-(Q12-B): track 13.1 -> 15.0 mm
- net Net-(Q11-C): track 29.3 -> 27.4 mm
- net Net-(Q3-E): track 6.16 -> 4.50 mm
- net Net-(Q7-E): track 9.17 -> 7.85 mm
- net Net-(Q4-C): track 22.8 -> 24.0 mm
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