File: main/main.kicad_sch (KiCad schematic)
At the start: 36 parts, among them J102 Conn_01x08_Socket, U105 TL072, U106 TL072

Commit message: wip
Parts:
- removed C103, C104, C105, C106, C107, C108: 100n, Capacitor_THT:C_Disc_D4.3mm_W1.9mm_P5.00mm, symbol Device:C
- removed C110, C111, C112, C113: C_Polarized_US, Capacitor_THT:CP_Radial_D6.3mm_P2.50mm, symbol Device:C_Polarized_US
- removed D101, D102, D106, D107: BAT51, Diode_THT:D_DO-15_P12.70mm_Horizontal, symbol Device:D_Schottky
- removed D104, D105, D108, D109: D_Schottky, Diode_THT:D_DO-15_P12.70mm_Horizontal, symbol Device:D_Schottky
- removed J102: Conn_01x08_Socket, Connector_Molex:Molex_KK-254_AE-6410-08A_1x08_P2.54mm_Vertical, symbol Connector:Conn_01x08_Socket
- removed R102, R105, R106, R109, R110, R111, R112, R113, R114, R115: 4k7, Resistor_THT:R_Axial_DIN0207_L6.3mm_D2.5mm_P10.16mm_Horizontal, symbol Device:R_US
- removed R103, R104: 100, Resistor_THT:R_Axial_DIN0207_L6.3mm_D2.5mm_P10.16mm_Horizontal, symbol Device:R_US
- removed RV101, RV102, RV103: R_Potentiometer_Trim_US, Potentiometer_THT:Potentiometer_Bourns_3296W_Vertical, symbol Device:R_Potentiometer_Trim_US
- removed U105, U106: TL072, Package_DIP:DIP-8_W7.62mm_LongPads, symbol Amplifier_Operational:TL072
